File: schematics/cpe/cpe_comb.kicad_sch (KiCad schematic)
At the start: 18 parts

Commit message: update schematics to include switchboxes
Parts:
- renumbered U49 to U1960
Connections:
- new net: M30.D0, U1960., U52.
- new net: M30.S, U1960., U65., U66.
- new net: M31.S, U58., U64., U65.
