File: schematics/cpe/cpe_comb_addf2.kicad_sch (KiCad schematic)
At the start: 18 parts

Commit message: further CPE schematic updates
Parts:
- removed INIT_L4, INIT_L5, INIT_L6, L8: ~, symbol peppercorn:LUT2 with C_I mux
- removed L10, L11, L9: ~, symbol peppercorn:LUT2
- removed M30, M31: ~, symbol peppercorn:MUX2
- removed U49, U64, U66: ~, symbol peppercorn:XOR
- removed U52, U53: ~, symbol peppercorn:AND
- removed U54: ~, symbol peppercorn:AO21
- removed U56: ~, symbol peppercorn:XNOR
- removed U58: ~, symbol peppercorn:XOR3
- removed U65: ~, symbol peppercorn:OR
- added C6: ~, symbol peppercorn:MUX2B
- added INIT_L12, INIT_L13, INIT_L14, L16: ~, symbol peppercorn:LUT2 with C_I mux
- added L17, L18, L19: ~, symbol peppercorn:LUT2
- added M14, M15: ~, symbol peppercorn:MUX2 (conceptual)
- added M20, M21: ~, symbol peppercorn:MUX2
- added U10, U11: ~, symbol peppercorn:AND
- added U36, U47: ~, symbol peppercorn:OR
- added U38: ~, symbol peppercorn:NAND
- added U39, U43: ~, symbol peppercorn:XOR3
- added U42, U46, U48: ~, symbol peppercorn:XOR
Connections:
- net CADD_A: now also M14.Y
- net CADD_S: now also U38.
- net CINX: now also C6.D1, INIT_L12.D1
- net CINY1: now also C6.D0, U39.
- net CINY2: now also M21.D0, U46.
- net COMB1OUT: now also L19.Y
- net COMB2OUT: now also U42.
- net COY2_S: now also U47.
- net COY2_a: now also M20.Y
- net IN1: now also L16.D0
- net IN2: now also L16.D0
- net IN3: now also INIT_L12.D0
- net IN4: now also INIT_L12.D0
- net IN5: now also INIT_L13.D0, U10.
- net IN6: now also INIT_L13.D0
- net IN7: now also INIT_L14.D0
- net IN8: now also INIT_L14.D0, U11.
- net L00: now also L16.Y, L17.D0, U36.
- net L01: now also INIT_L12.Y, L17.D1, U36.
- net L02: now also INIT_L13.Y, L18.D0, M14.D1, M15.D0
- net L11: now also L18.Y, L19.D1, M15.S, U38., U39.
- net MULTO1: now also U46.
- net MULTO2: now also U48.
- net PINX: now also INIT_L14.D1
- net PINY1: now also INIT_L13.D1, L16.D1
- net PINY2: now also U10., U11.
- new net: M20.D1, M21.D1, U11., U39.
- new net: M21.S, U39., U46., U47.
- new net: M20.D0, U10., U43.
- new net: M15.Y, U42., U43.
- new net: M20.S, U43., U47., U48.
- new net: INIT_L14.Y, L18.D1
- new net: M14.D0, U36.
- new net: M21.Y, U48.
- new net CIN: C6.Y, M15.D1
- new net L10: L17.Y, L19.D0, M14.S, U38., U42., U43.
Other:
- note added: "C_FUNCTION = 2: ADDF2 This provides a 2-bit full adder. The addition is performed in propagate/generate style. C_FUNCTION = 3: MULT This provides a 2x2-bit Booth multiplier. The dedicated logic performs multiplication by B[1], while multiplication by B[0] is performed within the soft logic. (These functions differ by how they set up the downstream carry and propagation lines; from this part of th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"
- note added: "C_HORIZ"
- note added: "In multiplier mode, the LUTs should be set up as: L10 = (A[1] & B[0]) ^ SI[1] L11 = (A[0] & B[0]) ^ SI[0]"
- title: CPE: Default Mode -> CPE: 2-bit Adder/Multiplier Mode

Commit message: update CPE schematics to cover C/P lines
Connections:
- new net: M21.S, U39., U46., U47.
- new net: M20.D0, U10., U43.
- new net: M15.Y, U42., U43.
- new net: M20.S, U43., U47., U48.
Other:
- note added: "C_FUNCTION = 2: ADDF2 This provides a 2-bit full adder. The addition is performed in propagate/generate style. Setting C_HORIZ configures the adder to propagate carries horizontally, rather than vertically. This feature isn't implemented in p_r or nextpnr because horizontal carries have twice the propagation delay of vertical carries. C_FUNCTION = 3: MULT This provides a 2x2-bit Booth multiplier.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"
- note removed: "C_FUNCTION = 2: ADDF2 This provides a 2-bit full adder. The addition is performed in propagate/generate style. C_FUNCTION = 3: MULT This provides a 2x2-bit Booth multiplier. The dedicated logic performs multiplication by B[1], while multiplication by B[0] is performed within the soft logic. (These functions differ by how they set up the downstream carry and propagation lines; from this part of th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"
Changed lines of the file:
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@@
 		)
 	)
-	(text "C_FUNCTION = 2: ADDF2\n\nThis provides a 2-bit full adder.\n\nThe addition is performed in propagate/generate style.\n\nC_FUNCTION = 3: MULT\n\nThis provides a 2x2-bit Booth multiplier.\n\nThe dedicated logic performs multiplication by B[1], while\nmultiplication by B[0] is performed within the soft logic.\n\n(These functions differ by how they set up the downstream\ncarry and propagation lines; from this part of the logic\nthey function identically, thus have been grouped together)"
+	(text "C_FUNCTION = 2: ADDF2\n\nThis provides a 2-bit full adder.\n\nThe addition is performed in propagate/generate style.\n\nSetting C_HORIZ configures the adder to propagate carries\nhorizontally, rather than vertically. This feature isn't\nimplemented in p_r or nextpnr because horizontal carries\nhave twice the propagation delay of vertical carries.\n\nC_FUNCTION = 3: MULT\n\nThis provides a 2x2-bit Booth multiplier.\n\nThe dedicated logic performs multiplication by B[1], while\nmultiplication by B[0] is performed within the soft logic.\n\n(These functions differ by how they set up the downstream\ncarry and propagation lines; from this part of the logic\nthey function identically, thus have been grouped together)"
 		(exclude_from_sim no)
 		(at 76.2 177.8 0)

Commit message: update schematics to include switchboxes
Connections:
- new net: M21.S, U39., U46., U47.
- new net: M20.D0, U10., U43.
- new net: M15.Y, U42., U43.
- new net: M20.S, U43., U47., U48.
