File: schematics/cpe/prjpeppercorn.kicad_sch (KiCad schematic)
At the start: 0 parts

Commit message: update schematics to include switchboxes
Other:
- sheet Cologne Processing Element renamed CPE11
- added sheet Big Switch Box (sb_big.kicad_sch)
- added sheet Big Switch Box1 (sb_big.kicad_sch)
- added sheet Big Switch Box2 (sb_big.kicad_sch)
- added sheet Big Switch Box3 (sb_big.kicad_sch)
- added sheet CPE12 (cpe.kicad_sch)
- added sheet CPE21 (cpe.kicad_sch)
- added sheet CPE22 (cpe.kicad_sch)
- added sheet Cologne Processing Element10 (cpe.kicad_sch)
- added sheet Cologne Processing Element11 (cpe.kicad_sch)
- added sheet Cologne Processing Element12 (cpe.kicad_sch)
- added sheet Cologne Processing Element13 (cpe.kicad_sch)
- added sheet Cologne Processing Element14 (cpe.kicad_sch)
- added sheet Cologne Processing Element15 (cpe.kicad_sch)
- added sheet Cologne Processing Element4 (cpe.kicad_sch)
- added sheet Cologne Processing Element5 (cpe.kicad_sch)
- added sheet Cologne Processing Element6 (cpe.kicad_sch)
- added sheet Cologne Processing Element7 (cpe.kicad_sch)
- added sheet Cologne Processing Element8 (cpe.kicad_sch)
- added sheet Cologne Processing Element9 (cpe.kicad_sch)
- added sheet Input Multiplexer (im.kicad_sch)
- added sheet Input Multiplexer1 (im.kicad_sch)
- added sheet Input Multiplexer10 (im.kicad_sch)
- added sheet Input Multiplexer11 (im.kicad_sch)
- added sheet Input Multiplexer12 (im.kicad_sch)
- added sheet Input Multiplexer13 (im.kicad_sch)
- added sheet Input Multiplexer14 (im.kicad_sch)
- added sheet Input Multiplexer15 (im.kicad_sch)
- added sheet Input Multiplexer2 (im.kicad_sch)
- added sheet Input Multiplexer3 (im.kicad_sch)
- added sheet Input Multiplexer4 (im.kicad_sch)
- added sheet Input Multiplexer5 (im.kicad_sch)
- added sheet Input Multiplexer6 (im.kicad_sch)
- added sheet Input Multiplexer7 (im.kicad_sch)
- added sheet Input Multiplexer8 (im.kicad_sch)
- added sheet Input Multiplexer9 (im.kicad_sch)
- added sheet Output Multiplexer (1,1) (om11.kicad_sch)
- added sheet Output Multiplexer (1,1)1 (om11.kicad_sch)
- added sheet Output Multiplexer (1,1)2 (om11.kicad_sch)
- added sheet Output Multiplexer (1,1)3 (om11.kicad_sch)
- added sheet Output Multiplexer (2,2) (om22.kicad_sch)
- added sheet Output Multiplexer (2,2)1 (om22.kicad_sch)
- added sheet Output Multiplexer (2,2)2 (om22.kicad_sch)
- added sheet Output Multiplexer (2,2)3 (om22.kicad_sch)
- added sheet Small Switch Box (sb_sml.kicad_sch)
- added sheet Small Switch Box1 (sb_sml.kicad_sch)
- added sheet Small Switch Box2 (sb_sml.kicad_sch)
- added sheet Small Switch Box3 (sb_sml.kicad_sch)
- sheet CPE11 ports: added IN1, OUT1, OUT2; removed none
- note added: "FOUR-GROUP TYPE A"
- note added: "FOUR-GROUP TYPE B"
- note added: "Only Plane 1 is depicted for conciseness; in the switchbox sheets you can see the connections to other planes."
